Commit message: 10Dof urdf working.

File: resources/robots/kbot-headless-full-collisions/kbot_10dof.urdf (robot description, URDF)
Before this commit: robot kbotv2p0_headless, 23 links, 22 joints
Joints:
- joint dof_left_elbow_02: origin xyz=-0.018500 0.010000 0.137000 rpy=-3.141593 1.570796 0 -> xyz=-0.018500 0.010000 0.137000 rpy=1.570796 0 -1.570796
- joint dof_left_shoulder_roll_03: origin xyz=-0.024250 0 -0.080000 rpy=-3.141593 1.570796 0 -> xyz=-0.024250 0 -0.080000 rpy=1.57079821 1.3962634 -1.57079482
- joint dof_right_elbow_02: origin xyz=0.018500 -0.010000 -0.137000 rpy=0 1.570796 0 -> xyz=0.018500 -0.010000 -0.137000 rpy=-1.570796 0 -1.570796
- joint dof_right_shoulder_roll_03: origin xyz=-0.024250 0 -0.080000 rpy=-3.141593 -1.570796 0 -> xyz=-0.024250 0 -0.080000 rpy=-1.57079821 -1.3962634 -1.57079413
