Commit message: Updated urdfs to newest kbot.

File: resources/robots/kbot-headless-full-collisions/robot.urdf (robot description, URDF)
Before this commit: robot kbotv2p0_headless, 23 links, 22 joints
Links:
- removed link KB_C_501X_Left_Bayonet_Adapter_Hard_Stop
- removed link KB_C_501X_Right_Bayonet_Adapter_Hard_Stop
- removed link KB_D_501L_L_LEG_FOOT
- removed link KB_D_501R_R_LEG_FOOT
- removed link KC_C_104L_PitchHardstopDriven
- removed link KC_C_104R_PitchHardstopDriven
- removed link KC_C_202L
- removed link KC_C_401L_L_UpForearmDrive
- removed link KC_D_102L_L_Hip_Yoke_Drive
- removed link KC_D_102R_R_Hip_Yoke_Drive
- removed link KC_D_301L_L_Femur_Lower_Drive
- removed link KC_D_301R_R_Femur_Lower_Drive
- removed link KC_D_401L_L_Shin_Drive
- removed link KC_D_401R_R_Shin_Drive
- removed link RS03_5
- removed link RS03_6
- removed link Torso_Side_Right
- added link KC_C_101R_ShldYokeDrive, mass 0.569870; collision mesh filename=meshes/KC_C_101R_ShldYokeDrive.collision.stl; visual mesh filename=meshes/KC_C_101R_ShldYokeDrive.stl
- added link KC_C_401L_Up_Forearm_Drive, mass 0.641873; collision mesh filename=meshes/KC_C_401L_Up_Forearm_Drive.collision.stl; visual mesh filename=meshes/KC_C_401L_Up_Forearm_Drive.stl
- added link KD_C_101L_ShldYokeDrive, mass 0.569863; collision mesh filename=meshes/KD_C_101L_ShldYokeDrive.collision.stl; visual mesh filename=meshes/KD_C_101L_ShldYokeDrive.stl
- added link KD_C_301L_LowerBicepDrive, mass 0.866827; collision mesh filename=meshes/KD_C_301L_LowerBicepDrive.collision.stl; visual mesh filename=meshes/KD_C_301L_LowerBicepDrive.stl
- added link KD_D_101L_L_Hip_Static, mass 11.824875; collision mesh filename=meshes/KD_D_101L_L_Hip_Static.collision.stl; visual mesh filename=meshes/KD_D_101L_L_Hip_Static.stl
- added link KD_D_102L_L_Hip_Yoke_Drive, mass 0.550354; collision mesh filename=meshes/KD_D_102L_L_Hip_Yoke_Drive.collision.stl; visual mesh filename=meshes/KD_D_102L_L_Hip_Yoke_Drive.stl
- added link KD_D_102R, mass 0.550361; collision mesh filename=meshes/KD_D_102R.collision.stl; visual mesh filename=meshes/KD_D_102R.stl
- added link KD_D_301L_L_Femur_Lower_Drive, mass 2.349254; collision mesh filename=meshes/KD_D_301L_L_Femur_Lower_Drive.collision.stl; visual mesh filename=meshes/KD_D_301L_L_Femur_Lower_Drive.stl
- added link KD_D_301R, mass 2.349261; collision mesh filename=meshes/KD_D_301R.collision.stl; visual mesh filename=meshes/KD_D_301R.stl
- added link KD_D_401L_L_Shin_Drive, mass 1.684707; collision mesh filename=meshes/KD_D_401L_L_Shin_Drive.collision.stl; visual mesh filename=meshes/KD_D_401L_L_Shin_Drive.stl
- added link KD_D_401R, mass 1.684717; collision mesh filename=meshes/KD_D_401R.collision.stl; visual mesh filename=meshes/KD_D_401R.stl
- added link LFootBushing_GPF_1517_12, mass 0.608966; collision mesh filename=meshes/LFootBushing_GPF_1517_12.collision.stl; visual mesh filename=meshes/LFootBushing_GPF_1517_12.stl
- added link L_Hip_Roll_RS03, mass 2.396969; collision mesh filename=meshes/L_Hip_Roll_RS03.collision.stl; visual mesh filename=meshes/L_Hip_Roll_RS03.stl
- added link L_Hip_Roll_RS03_2, mass 2.396917; collision mesh filename=meshes/L_Hip_Roll_RS03_2.collision.stl; visual mesh filename=meshes/L_Hip_Roll_RS03_2.stl
- added link PRT0001, mass 0.462356; collision mesh filename=meshes/PRT0001.collision.stl; visual mesh filename=meshes/PRT0001.stl
- added link PRT0001_2, mass 0.462356; collision mesh filename=meshes/PRT0001_2.collision.stl; visual mesh filename=meshes/PRT0001_2.stl
- added link RFootBushing_GPF_1517_12, mass 0.608742; collision mesh filename=meshes/RFootBushing_GPF_1517_12.collision.stl; visual mesh filename=meshes/RFootBushing_GPF_1517_12.stl
- link KC_C_202R: mass 0.743508 -> 0.753224; geometry collision mesh filename=meshes/KC_C_202R.collision.stl; visual mesh filename=meshes/KC_C_202R.stl
- link KC_C_401R_R_UpForearmDrive: mass 0.585204 -> 0.641859; geometry collision mesh filename=meshes/KC_C_401R_R_UpForearmDrive.collision.stl; visual mesh filename=meshes/KC_C_401R_R_UpForearmDrive.stl
- link RS03_3: mass 1.676509 -> 1.789232; geometry collision mesh filename=meshes/RS03_3.collision.stl; visual mesh filename=meshes/RS03_3.stl
- link RS03_4: mass 2.373184 -> 1.789190; geometry collision mesh filename=meshes/RS03_4.collision.stl; visual mesh filename=meshes/RS03_4.stl
- link imu: geometry collision mesh filename=meshes/imu.collision.stl; visual mesh filename=meshes/imu.stl
Joints:
- joint base_joint: child Torso_Side_Right -> KD_D_101L_L_Hip_Static; origin xyz=0 -0.095 0 rpy=0 0 1.5708 -> xyz=0 0.035 0 rpy=0 0 1.5708
- joint dof_left_ankle_02: child KB_D_501L_L_LEG_FOOT -> LFootBushing_GPF_1517_12; limit lower=-1.256637 upper=0.226893 effort=17 velocity=37.699 -> lower=-1.134464 upper=0.261799 effort=17 velocity=37.699; origin xyz=-0.030000 -0.290000 0.035100 rpy=-3.141593 0 0 -> xyz=-0.030000 -0.290000 0.000950 rpy=3.141593 0 0; parent KC_D_401L_L_Shin_Drive -> KD_D_401L_L_Shin_Drive
- joint dof_left_elbow_02: axis 0 0 -1 -> 0 0 1; child KC_C_401L_L_UpForearmDrive -> KC_C_401L_Up_Forearm_Drive; origin xyz=-0.018500 0.010000 0.137000 rpy=-3.141593 1.570796 0 -> xyz=-0.019000 -0.010000 -0.137000 rpy=1.570796 0 1.570796; parent KC_C_202L -> KD_C_301L_LowerBicepDrive
- joint dof_left_hip_pitch_04: child KC_D_102L_L_Hip_Yoke_Drive -> KD_D_102L_L_Hip_Yoke_Drive; origin xyz=0.147969 0.000007 -0.284479 rpy=-1.570796 0 1.570796 -> xyz=0.030112 0.000852 -0.027644 rpy=-1.570796 0 1.570796; parent Torso_Side_Right -> KD_D_101L_L_Hip_Static
- joint dof_left_hip_roll_03: child RS03_5 -> L_Hip_Roll_RS03; origin xyz=-0.028250 0.030000 -0.071000 rpy=0 1.570796 0 -> xyz=-0.028250 0.030000 -0.071000 rpy=3.141593 -1.570796 0; parent KC_D_102L_L_Hip_Yoke_Drive -> KD_D_102L_L_Hip_Yoke_Drive
- joint dof_left_hip_yaw_03: axis 0 0 -1 -> 0 0 1; child KC_D_301L_L_Femur_Lower_Drive -> KD_D_301L_L_Femur_Lower_Drive; origin xyz=0 0.143000 0.024250 rpy=-1.570796 0 0 -> xyz=0 -0.143000 0.025250 rpy=1.570796 0 -3.141593; parent RS03_5 -> L_Hip_Roll_RS03
- joint dof_left_knee_04: child KC_D_401L_L_Shin_Drive -> KD_D_401L_L_Shin_Drive; origin xyz=-0.020500 -0.021000 0.212000 rpy=-1.570796 0 -1.570796 -> xyz=-0.021000 0.021000 -0.212000 rpy=1.570796 0 1.570796; parent KC_D_301L_L_Femur_Lower_Drive -> KD_D_301L_L_Femur_Lower_Drive
- joint dof_left_shoulder_pitch_03: axis 0 0 1 -> 0 0 -1; child KC_C_104L_PitchHardstopDriven -> KD_C_101L_ShldYokeDrive; limit lower=-1.396263 upper=3.141593 effort=60 velocity=18.849 -> lower=-1.047198 upper=3.490658 effort=60 velocity=18.849; origin xyz=0.213969 0.000007 0.126021 rpy=-1.570796 0 1.570796 -> xyz=0.095112 0.000852 0.382856 rpy=0 1.570796 0; parent Torso_Side_Right -> KD_D_101L_L_Hip_Static
- joint dof_left_shoulder_roll_03: child RS03_6 -> RS03_4; limit lower=-0.349066 upper=1.658063 effort=60 velocity=18.849 -> lower=-0.436332 upper=1.658063 effort=60 velocity=18.849; origin xyz=-0.024250 0 -0.080000 rpy=-3.141593 1.570796 0 -> xyz=0 -0.024250 0.080000 rpy=1.570796 -1.570796 0; parent KC_C_104L_PitchHardstopDriven -> KD_C_101L_ShldYokeDrive
- joint dof_left_shoulder_yaw_02: axis 0 0 -1 -> 0 0 1; child KC_C_202L -> KD_C_301L_LowerBicepDrive; limit lower=-1.658063 upper=1.658063 effort=17 velocity=37.699 -> lower=-1.671886 upper=1.671886 effort=17 velocity=37.699; origin xyz=0.013000 -0.142000 -0.030250 rpy=1.570796 0 0 -> xyz=0.013000 -0.142500 -0.030750 rpy=-1.570796 0 0; parent RS03_6 -> RS03_4
- joint dof_left_wrist_00: child KB_C_501X_Left_Bayonet_Adapter_Hard_Stop -> PRT0001_2; limit lower=-1.745329 upper=1.745329 effort=14 velocity=27.227 -> lower=-1.378810 upper=1.378810 effort=14 velocity=27.227; origin xyz=-0.103000 0.017350 -0.018000 rpy=-3.141593 1.570796 0 -> xyz=0.017350 -0.103000 0.018000 rpy=1.570796 -1.570796 0; parent KC_C_401L_L_UpForearmDrive -> KC_C_401L_Up_Forearm_Drive
- joint dof_right_ankle_02: axis 0 0 1 -> 0 0 -1; child KB_D_501R_R_LEG_FOOT -> RFootBushing_GPF_1517_12; limit lower=-0.226893 upper=1.256637 effort=17 velocity=37.699 -> lower=-0.261799 upper=1.134464 effort=17 velocity=37.699; origin xyz=-0.030000 0.290000 0.035100 rpy=0 0 0 -> xyz=-0.030000 -0.290000 -0.000950 rpy=0 0 0; parent KC_D_401R_R_Shin_Drive -> KD_D_401R
- joint dof_right_elbow_02: axis 0 0 -1 -> 0 0 1; origin xyz=0.018500 -0.010000 -0.137000 rpy=0 1.570796 0 -> xyz=0.019000 -0.010000 -0.137000 rpy=-1.570796 0 1.570796
- joint dof_right_hip_pitch_04: child KC_D_102R_R_Hip_Yoke_Drive -> KD_D_102R; origin xyz=0.037469 0.000007 -0.284479 rpy=1.570796 0 1.570796 -> xyz=-0.081888 0.000852 -0.027644 rpy=1.570796 0 1.570796; parent Torso_Side_Right -> KD_D_101L_L_Hip_Static
- joint dof_right_hip_roll_03: axis 0 0 -1 -> 0 0 1; child RS03_4 -> L_Hip_Roll_RS03_2; origin xyz=-0.028250 -0.030000 -0.071000 rpy=3.141593 -1.570796 0 -> xyz=-0.028250 -0.030000 -0.071000 rpy=0 -1.570796 0; parent KC_D_102R_R_Hip_Yoke_Drive -> KD_D_102R
- joint dof_right_hip_yaw_03: axis 0 0 -1 -> 0 0 1; child KC_D_301R_R_Femur_Lower_Drive -> KD_D_301R; origin xyz=0 0.143000 0.024250 rpy=-1.570796 0 0 -> xyz=0 -0.143000 -0.025250 rpy=-1.570796 0 0; parent RS03_4 -> L_Hip_Roll_RS03_2
- joint dof_right_knee_04: axis 0 0 1 -> 0 0 -1; child KC_D_401R_R_Shin_Drive -> KD_D_401R; origin xyz=0.020500 -0.021000 0.212000 rpy=1.570796 0 -1.570796 -> xyz=0.021000 0.021000 -0.212000 rpy=1.570796 0 1.570796; parent KC_D_301R_R_Femur_Lower_Drive -> KD_D_301R
- joint dof_right_shoulder_pitch_03: axis 0 0 1 -> 0 0 -1; child KC_C_104R_PitchHardstopDriven -> KC_C_101R_ShldYokeDrive; limit lower=-3.141593 upper=1.396263 effort=60 velocity=18.849 -> lower=-3.490658 upper=1.047198 effort=60 velocity=18.849; origin xyz=-0.028031 0.000007 0.126021 rpy=1.570796 0 1.570796 -> xyz=-0.146888 0.000852 0.382856 rpy=0 -1.570796 0; parent Torso_Side_Right -> KD_D_101L_L_Hip_Static
- joint dof_right_shoulder_roll_03: axis 0 0 -1 -> 0 0 1; limit lower=-1.658063 upper=0.349066 effort=60 velocity=18.849 -> lower=-1.658063 upper=0.436332 effort=60 velocity=18.849; origin xyz=-0.024250 0 -0.080000 rpy=-3.141593 -1.570796 0 -> xyz=0 -0.024250 0.080000 rpy=1.570796 1.570796 0; parent KC_C_104R_PitchHardstopDriven -> KC_C_101R_ShldYokeDrive
- joint dof_right_shoulder_yaw_02: limit lower=-1.658063 upper=1.658063 effort=17 velocity=37.699 -> lower=-1.671886 upper=1.671886 effort=17 velocity=37.699; origin xyz=-0.013000 0.142000 0.030250 rpy=1.570796 0 0 -> xyz=-0.013000 -0.142500 -0.031670 rpy=-1.570796 0 0
- joint dof_right_wrist_00: axis 0 0 1 -> 0 0 -1; child KB_C_501X_Right_Bayonet_Adapter_Hard_Stop -> PRT0001; limit lower=-1.745329 upper=1.745329 effort=14 velocity=27.227 -> lower=-1.378810 upper=1.378810 effort=14 velocity=27.227; origin xyz=0.103000 0.017350 -0.018000 rpy=0 -1.570796 0 -> xyz=0.017350 0.103000 0.018000 rpy=-1.570796 1.570796 0
- joint frame_imu_site: origin xyz=0.093118 -0.000341 0.188248 rpy=0 0 -1.570796 -> xyz=-0.025422 -0.001897 0.440523 rpy=0 0 0; parent Torso_Side_Right -> KD_D_101L_L_Hip_Static

File: resources/robots/kbot-headless/robot.urdf (robot description, URDF)
Before this commit: robot assy_forurdf, 23 links, 22 joints
Joints:
- joint dof_left_ankle_02: limit lower=-1.134464 upper=0.261799 effort=15 velocity=37.699 -> lower=-1.134464 upper=0.261799 effort=17 velocity=37.699
- joint dof_right_ankle_02: limit lower=-0.261799 upper=1.134464 effort=15 velocity=37.699 -> lower=-0.261799 upper=1.134464 effort=17 velocity=37.699
