Commit message: Updated to the newest kbot urdf.

File: resources/robots/kbot-headless/robot.urdf (robot description, URDF)
Before this commit: robot kd_headless, 23 links, 22 joints
Links:
- link KD_D_101L_L_Hip_Static: mass 12.606875 -> 11.824875
- link LFootBushing_GPF_1517_12: geometry collision mesh filename=meshes/LFootBushing_GPF_1517_12.collision.stl; visual mesh filename=meshes/LFootBushing_GPF_1517_12.stl
- link RFootBushing_GPF_1517_12: geometry collision mesh filename=meshes/RFootBushing_GPF_1517_12.collision.stl; visual mesh filename=meshes/RFootBushing_GPF_1517_12.stl
- link RS03_4: mass 1.789191 -> 1.789190
Joints:
- joint dof_left_ankle_02: limit lower=-1.134464 upper=0.261799 effort=17 velocity=37.699 -> lower=-1.134464 upper=0.261799 effort=15 velocity=37.699
- joint dof_right_ankle_02: limit lower=-0.261799 upper=1.134464 effort=17 velocity=37.699 -> lower=-0.261799 upper=1.134464 effort=15 velocity=37.699
